File: 007_R00.kicad_pcb (KiCad board)
At the start: 2 copper layers, 99.1 x 78.7 mm, 14 parts, among them J1 CONN_02X28, SW1 SAVE, SW2 RESET, U1 74LS10, U2 2716, U3 74LS74, U4 74LS27

Commit message: Add files via upload
Parts:
- R1: footprint Resistors_THT:R_Axial_DIN0204_L3.6mm_D1.6mm_P7.62mm_Horizontal -> SINCLAIR:R_Axial_DIN0204_L3.6mm_D1.6mm_P11.43mm_Horizontal
Connections:
- net Net-(J1-Pad36) renamed /RD
Routing:
- net /ROMCS: track 73.0 -> 79.4 mm
- net Net-(D2-Pad2): track 26.2 -> 28.1 mm

Commit message: with edge conector
Parts:
- added ?: Symbol_CC-Attribution_CopperTop_Small, Symbols:Symbol_CC-Attribution_CopperTop_Small, F.Cu at (128.3, 104.8)
- added ?: Symbol_CC-Noncommercial_CopperTop_Small, Symbols:Symbol_CC-Noncommercial_CopperTop_Small, F.Cu at (134.6, 104.8)
- added ?: Symbol_CreativeCommons_CopperTop_Type2_Small, Symbols:Symbol_CreativeCommons_CopperTop_Type2_Small, F.Cu at (121.9, 104.8)
- added ?: Symbol_CC-ShareAlike_CopperTop_Small, Symbols:Symbol_CC-ShareAlike_CopperTop_Small, F.Cu at (141.0, 104.8)
- added REF***: OSHW-Symbol_6.7x6mm_SilkScreen, Symbols:OSHW-Symbol_6.7x6mm_SilkScreen, F.Cu at (137.2, 113.0)
- C2: footprint Capacitors_THT:CP_Axial_L10.0mm_D6.0mm_P15.00mm_Horizontal -> Capacitors_THT:CP_Radial_D6.3mm_P2.50mm
- moved C2 5.72 mm to (168.9, 86.4)
- moved SW2 2.54 mm to (174.0, 119.4)
- moved C1 2.54 mm to (175.3, 85.1)
Routing:
- net Net-(C1-Pad1): track 71.1 -> 67.5 mm
- net GND: track 279.9 -> 281.9 mm
- net /RESET: track 138.7 -> 137.4 mm
- net (no net): track 23.5 -> 22.9 mm
Other:
- board size 99.1 x 78.7 mm -> 99.1 x 73.7 mm
- board text added: "2017 Alvaro Alea for VdR"
