File: 007_R00.sch (KiCad schematic (older format))
At the start: 14 parts, among them J1 CONN_02X28, SW1 SAVE, SW2 RESET, U1 74LS10, U2 2716, U3 74LS74, U4 74LS27

Commit message: Add files via upload
Connections:
- net labels added: RD
Changed lines of the file:
@@
 F 3 "" H 8950 6050 50  0001 C CNN
 	1    8950 6050
-	1    0    0    -1
+	-1   0    0    1
 $EndComp
 $Comp
@@
 Wire Wire Line
 	5950 2750 5950 3300
+Text Label 2700 2750 0    60   ~ 0
+RD
 $EndSCHEMATC

Commit message: with edge conector
Parts:
- R1: MOUSER PART (none) -> 791-RC1/4-331JB
- R2: MOUSER PART (none) -> 791-RC1/4-101JB
- R3: MOUSER PART (none) -> 791-RC1/4-472JB
- U1: MOUSER PART (none) -> 595-SN74LS10N
- U3: MOUSER PART (none) -> 595-SN74LS74AN
- U4: MOUSER PART (none) -> 595-SN74LS27N
Changed lines of the file:
@@
 F 2 "Housings_DIP:DIP-14_W7.62mm_LongPads" H 8300 4950 50  0001 C CNN
 F 3 "" H 8300 4950 50  0001 C CNN
+F 4 "595-SN74LS10N" H 8300 4950 60  0001 C CNN "MOUSER PART"
 	1    8300 4950
 	1    0    0    -1
@@
 F 2 "Housings_DIP:DIP-14_W7.62mm_LongPads" H 5900 5700 50  0001 C CNN
 F 3 "" H 5900 5700 50  0001 C CNN
+F 4 "595-SN74LS74AN" H 5900 5700 60  0001 C CNN "MOUSER PART"
 	1    5900 5700
 	1    0    0    -1
@@
 F 2 "Housings_DIP:DIP-14_W7.62mm_LongPads" H 7450 6050 50  0001 C CNN
 F 3 "" H 7450 6050 50  0001 C CNN
+F 4 "595-SN74LS27N" H 7450 6050 60  0001 C CNN "MOUSER PART"
 	3    7450 6050
 	1    0    0    -1
@@
 F 2 "Resistors_THT:R_Axial_DIN0204_L3.6mm_D1.6mm_P7.62mm_Horizontal" V 7180 4700 50  0001 C CNN
 F 3 "" H 7250 4700 50  0001 C CNN
+F 4 "791-RC1/4-101JB" V 7250 4700 60  0001 C CNN "MOUSER PART"
 	1    7250 4700
 	1    0    0    -1
@@
 F 2 "Resistors_THT:R_Axial_DIN0204_L3.6mm_D1.6mm_P7.62mm_Horizontal" V 3980 4500 50  0001 C CNN
 F 3 "" H 4050 4500 50  0001 C CNN
+F 4 "791-RC1/4-472JB" V 4050 4500 60  0001 C CNN "MOUSER PART"
 	1    4050 4500
 	1    0    0    -1
@@
 F 2 "Resistors_THT:R_Axial_DIN0204_L3.6mm_D1.6mm_P7.62mm_Horizontal" V 8530 5850 50  0001 C CNN
 F 3 "" H 8600 5850 50  0001 C CNN
+F 4 "791-RC1/4-331JB" V 8600 5850 60  0001 C CNN "MOUSER PART"
 	1    8600 5850
 	1    0    0    -1
