File: 007_mini/007_mini.kicad_pcb (KiCad board)
At the start: 2 copper layers, 53.3 x 73.7 mm, 22 parts, among them J1 ZX_Spectrum_Connector_48K, SW1 SAVE, SW2 RESET, SW3 SW_DIP_x02, U1 2764, U2 74LS27, U3 74LS10, U5 74LS74

Commit message: mini pcb
Parts:
- moved C3 4.98 mm to (124.3, 72.9), turned to 180 degrees
Routing:
- net GND: track 226.7 -> 207.3 mm
- net Net-(D2-Pad2): track 44.8 -> 48.8 mm
- net +5V: track 170.6 -> 169.3 mm
Changed lines of the file:
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@@
     (thickness 1.6)
     (drawings 15)
-    (tracks 557)
+    (tracks 558)
     (zones 0)
     (modules 22)
@@
   )
   (module Capacitor_THT:C_Disc_D4.7mm_W2.5mm_P5.00mm (layer F.Cu)
-    (at 119.38 72.39)
+    (at 124.333 72.898 180)
     (descr "C, Disc series, Radial, pin pitch=5.00mm, diameter*width=4.7*2.5mm^2, Capacitor, http://www.vishay.com/docs/45233/krseries.pdf")
     (tags "C Disc series Radial pin pitch 5.00mm  diameter 4.7mm width 2.5mm Capacitor")
-    (fp_text reference C3 (at 7.62 0) (layer F.SilkS)
-      (effects (font (size 1 1) (thickness 0.15)))
-    )
-    (fp_text value 100n (at 2.5 2.56) (layer F.Fab)
+    (fp_text reference C3 (at 7.62 0 180) (layer F.SilkS)
+      (effects (font (size 1 1) (thickness 0.15)))
+    )
+    (fp_text value 100n (at 2.5 2.56 180) (layer F.Fab)
       (effects (font (size 1 1) (thickness 0.15)))
     )
@@
     (fp_line (start 6.05 1.6) (end 6.05 -1.6) (layer F.CrtYd) (width 0.05))
     (fp_line (start 6.05 -1.6) (end -1.05 -1.6) (layer F.CrtYd) (width 0.05))
-    (fp_text user %R (at 2.5 0) (layer F.Fab)
-      (effects (font (size 1 1) (thickness 0.15)))
-    )
-    (pad 1 thru_hole circle (at 0 0) (size 1.6 1.6) (drill 0.8) (layers *.Cu *.Mask)
+    (fp_text user %R (at 2.5 0 180) (layer F.Fab)
+      (effects (font (size 1 1) (thickness 0.15)))
+    )
+    (pad 1 thru_hole circle (at 0 0 180) (size 1.6 1.6) (drill 0.8) (layers *.Cu *.Mask)
       (net 12 +5V))
-    (pad 2 thru_hole circle (at 5 0) (size 1.6 1.6) (drill 0.8) (layers *.Cu *.Mask)
+    (pad 2 thru_hole circle (at 5 0 180) (size 1.6 1.6) (drill 0.8) (layers *.Cu *.Mask)
       (net 1 GND))
     (model ${KISYS3DMOD}/Capacitor_THT.3dshapes/C_Disc_D4.7mm_W2.5mm_P5.00mm.wrl
@@
   (segment (start 124.38 96.52) (end 124.354 96.5465) (width 0.762) (layer B.Cu) (net 1))
   (segment (start 124.354 96.5465) (end 124.354 96.5997) (width 0.762) (layer B.Cu) (net 1))
-  (segment (start 126.942 69.8275) (end 124.38 72.39) (width 0.762) (layer B.Cu) (net 1))
-  (segment (start 110.49 62.23) (end 112.325 62.23) (width 0.762) (layer B.Cu) (net 1))
-  (segment (start 112.325 62.23) (end 112.325 63.9428) (width 0.762) (layer B.Cu) (net 1))
   (segment (start 130.81 59.69) (end 132.095 59.69) (width 0.762) (layer B.Cu) (net 1))
   (segment (start 132.095 59.69) (end 135.31 59.69) (width 0.762) (layer B.Cu) (net 1))
@@
   (via (at 109.696 98.2589) (size 1.2) (layers F.Cu B.Cu) (net 1))
   (segment (start 128.618 97.4981) (end 135.382 95.25) (width 0.762) (layer B.Cu) (net 1))
-  (segment (start 124.38 72.39) (end 127.682 69.088) (width 0.762) (layer B.Cu) (net 1))
   (segment (start 131.079 69.088) (end 132.095 68.072) (width 0.762) (layer B.Cu) (net 1))
-  (segment (start 127.682 69.088) (end 131.079 69.088) (width 0.762) (layer B.Cu) (net 1))
   (segment (start 132.095 59.69) (end 132.095 68.072) (width 0.762) (layer B.Cu) (net 1))
   (segment (start 134.446 76.28) (end 135.382 77.216) (width 0.762) (layer B.Cu) (net 1))
@@
   (segment (start 136.779 58.221) (end 135.31 59.69) (width 0.762) (layer B.Cu) (net 1))
   (segment (start 136.779 52.07) (end 136.779 58.221) (width 0.762) (layer B.Cu) (net 1))
-  (segment (start 117.602 73.152) (end 117.602 69.219461) (width 0.762) (layer B.Cu) (net 1))
-  (segment (start 112.325 63.9428) (end 117.602 69.219461) (width 0.762) (layer B.Cu) (net 1))
-  (segment (start 121.609 74.041) (end 118.491 74.041) (width 0.762) (layer B.Cu) (net 1))
   (segment (start 125.73 76.2) (end 123.768 76.2) (width 0.762) (layer B.Cu) (net 1))
   (segment (start 123.768 76.2) (end 121.609 74.041) (width 0.762) (layer B.Cu) (net 1))
-  (segment (start 118.491 74.041) (end 117.602 73.152) (width 0.762) (layer B.Cu) (net 1))
-  (segment (start 118.486539 70.104) (end 117.602 69.219461) (width 0.762) (layer B.Cu) (net 1))
-  (segment (start 122.094 70.104) (end 118.486539 70.104) (width 0.762) (layer B.Cu) (net 1))
-  (segment (start 124.38 72.39) (end 122.094 70.104) (width 0.762) (layer B.Cu) (net 1))
+  (segment (start 119.34463 74.041) (end 119.38 74.041) (width 0.762) (layer B.Cu) (net 1))
+  (segment (start 119.333 74.02937) (end 119.34463 74.041) (width 0.762) (layer B.Cu) (net 1))
+  (segment (start 119.333 72.898) (end 119.333 74.02937) (width 0.762) (layer B.Cu) (net 1))
+  (segment (start 121.609 74.041) (end 119.38 74.041) (width 0.762) (layer B.Cu) (net 1))
+  (segment (start 119.38 74.041) (end 118.491 74.041) (width 0.762) (layer B.Cu) (net 1))
+  (segment (start 110.89 62.23) (end 110.49 62.23) (width 0.762) (layer B.Cu) (net 1))
+  (segment (start 110.89 62.23) (end 114.808 66.148) (width 0.762) (layer B.Cu) (net 1))
+  (segment (start 114.808 70.358) (end 118.491 74.041) (width 0.762) (layer B.Cu) (net 1))
+  (segment (start 114.808 66.148) (end 114.808 70.358) (width 0.762) (layer B.Cu) (net 1))
   (segment (start 95.25 62.23) (end 93.5835 63.8965) (width 0.508) (layer F.Cu) (net 2))
   (segment (start 93.5835 63.8965) (end 93.5835 65.2781) (width 0.508) (layer F.Cu) (net 2))
@@
   (segment (start 114.338 104.102) (end 118.11 100.33) (width 0.508) (layer F.Cu) (net 10))
   (segment (start 99.06 110.49) (end 99.06 107.95) (width 0.508) (layer F.Cu) (net 11))
-  (segment (start 118.11 76.2) (end 116.402 76.2) (width 0.508) (layer F.Cu) (net 11))
-  (segment (start 116.402 76.2) (end 114.119 78.4832) (width 0.508) (layer F.Cu) (net 11))
-  (segment (start 114.119 78.4832) (end 114.119 95.3269) (width 0.508) (layer F.Cu) (net 11))
-  (segment (start 114.119 95.3269) (end 110.132 99.3132) (width 0.508) (layer F.Cu) (net 11))
-  (segment (start 110.132 99.3132) (end 108.598 99.3132) (width 0.508) (layer F.Cu) (net 11))
-  (segment (start 108.598 99.3132) (end 100.368 107.544) (width 0.508) (layer F.Cu) (net 11))
-  (segment (start 100.368 107.544) (end 100.368 107.95) (width 0.508) (layer F.Cu) (net 11))
-  (segment (start 100.368 107.95) (end 99.06 107.95) (width 0.508) (layer F.Cu) (net 11))
+  (segment (start 116.402 76.2) (end 118.11 76.2) (width 0.508) (layer F.Cu) (net 11))
+  (segment (start 114.119 96.447) (end 114.119 78.4832) (width 0.508) (layer F.Cu) (net 11))
+  (segment (start 99.06 107.95) (end 101.092 107.95) (width 0.508) (layer F.Cu) (net 11))
+  (segment (start 114.119 78.4832) (end 116.402 76.2) (width 0.508) (layer F.Cu) (net 11))
+  (segment (start 101.092 107.95) (end 103.378 105.664) (width 0.508) (layer F.Cu) (net 11))
+  (segment (start 103.378 105.664) (end 103.378 99.568) (width 0.508) (layer F.Cu) (net 11))
+  (segment (start 103.378 99.568) (end 105.791 97.155) (width 0.508) (layer F.Cu) (net 11))
+  (segment (start 105.791 97.155) (end 113.411 97.155) (width 0.508) (layer F.Cu) (net 11))
+  (segment (start 113.411 97.155) (end 114.119 96.447) (width 0.508) (layer F.Cu) (net 11))
   (segment (start 90.805 57.15) (end 91.1364 57.15) (width 0.762) (layer B.Cu) (net 12))
   (segment (start 91.1364 57.15) (end 92.0424 56.244) (width 0.762) (layer B.Cu) (net 12))
@@
   (segment (start 119.38 96.52) (end 113.03 102.87) (width 0.762) (layer F.Cu) (net 12))
   (segment (start 113.03 102.87) (end 106.68 102.87) (width 0.762) (layer F.Cu) (net 12))
-  (segment (start 106.68 102.87) (end 105.296 104.254) (width 0.762) (layer F.Cu) (net 12))
-  (segment (start 105.296 104.254) (end 105.296 109.106) (width 0.762) (layer F.Cu) (net 12))
-  (segment (start 105.296 109.106) (end 106.68 110.49) (width 0.762) (layer F.Cu) (net 12))
   (segment (start 109.22 110.49) (end 106.68 110.49) (width 0.762) (layer F.Cu) (net 12))
-  (segment (start 119.38 72.39) (end 116.113 69.1234) (width 0.762) (layer F.Cu) (net 12))
   (segment (start 116.113 61.5034) (end 110.49 55.88) (width 0.762) (layer F.Cu) (net 12))
   (segment (start 95.25 95.25) (end 98.296 95.25) (width 0.762) (layer B.Cu) (net 12))
@@
   (segment (start 116.148 67.31) (end 116.113 67.31) (width 0.762) (layer F.Cu) (net 12))
   (segment (start 118.11 67.31) (end 116.148 67.31) (width 0.762) (layer F.Cu) (net 12))
-  (segment (start 116.113 69.1234) (end 116.113 67.31) (width 0.762) (layer F.Cu) (net 12))
   (segment (start 116.113 67.31) (end 116.113 61.5034) (width 0.762) (layer F.Cu) (net 12))
   (segment (start 116.148 115.57) (end 115.951 115.767) (width 0.762) (layer F.Cu) (net 12))
@@
   (segment (start 118.11 95.25) (end 119.38 96.52) (width 0.762) (layer B.Cu) (net 12))
   (segment (start 118.11 91.44) (end 118.11 95.25) (width 0.762) (layer B.Cu) (net 12))
-  (segment (start 122.0209 72.39) (end 123.444 73.8131) (width 0.762) (layer B.Cu) (net 12))
-  (segment (start 119.38 72.39) (end 122.0209 72.39) (width 0.762) (layer B.Cu) (net 12))
-  (segment (start 128.117 73.8131) (end 123.444 73.8131) (width 0.762) (layer B.Cu) (net 12))
+  (segment (start 125.2481 73.8131) (end 124.333 72.898) (width 0.762) (layer B.Cu) (net 12))
+  (segment (start 128.117 73.8131) (end 125.2481 73.8131) (width 0.762) (layer B.Cu) (net 12))
+  (segment (start 118.745 67.31) (end 118.11 67.31) (width 0.762) (layer B.Cu) (net 12))
+  (segment (start 124.333 72.898) (end 118.745 67.31) (width 0.762) (layer B.Cu) (net 12))
+  (segment (start 105.664 110.49) (end 106.68 110.49) (width 0.762) (layer F.Cu) (net 12))
+  (segment (start 105.690051 102.87) (end 105.664 102.896051) (width 0.762) (layer F.Cu) (net 12))
+  (segment (start 105.637949 102.896051) (end 104.648 103.886) (width 0.762) (layer F.Cu) (net 12))
+  (segment (start 105.664 102.896051) (end 105.637949 102.896051) (width 0.762) (layer F.Cu) (net 12))
+  (segment (start 106.68 102.87) (end 105.690051 102.87) (width 0.762) (layer F.Cu) (net 12))
+  (segment (start 104.648 103.886) (end 104.648 109.474) (width 0.762) (layer F.Cu) (net 12))
+  (segment (start 104.648 109.474) (end 105.664 110.49) (width 0.762) (layer F.Cu) (net 12))
   (segment (start 87.63 52.07) (end 90.678 52.07) (width 0.508) (layer B.Cu) (net 13))
   (via (at 130.0226 87.8332) (size 1.2) (drill 0.4) (layers F.Cu B.Cu) (net 13))

Commit message: fix push buttons
Routing:
- net RESET: track 147.5 -> 160.0 mm
- net NMI: track 41.1 -> 45.3 mm
- net /A9: track 54.8 -> 59.0 mm
- net GND: track 207.3 -> 204.1 mm
- net /A11: track 54.6 -> 55.9 mm
- net Net-(U5-Pad12): track 10.2 -> 9.72 mm
